File: adcs_board/mcu.kicad_sch (KiCad schematic)
At the start: 23 parts, among them J1 Conn_01x04_Pin, J2 Conn_01x04_Pin, J3 Conn_01x04_Pin, J4 Conn_01x04_Pin, U1 STM32F103C8T6, U2 AMS1117-3.3, Y1 16 MHz

Commit message: adcs_board: resolve schematic ERC violations
- Corrected electrical rule check (ERC) errors in ADCS BDOT schematic
- Fixed unconnected pins and mismatched power nets
- Adjusted symbol properties for proper ERC compliance
- Ensured clean schematic validation with no remaining ERC issues
Parts:
- C1, C2: value 22u -> 22uF; footprint Capacitor_SMD:C_0805_2012Metric -> Capacitor_SMD:C_1206_3216Metric; Manufacturer (none) -> Samsung Electro-Mechanics; Manufacturer Part Number (none) -> CL31A226KAHNNNE
- C10, C6, C8, C9: value 100n -> 100nF; Manufacturer (none) -> Samsung Electro-Mechanics; Manufacturer Part Number (none) -> CL05B104KP5VPNC
- C11: value 10n -> 10nF; footprint Capacitor_SMD:C_0402_1005Metric -> Capacitor_SMD:C_0201_0603Metric; Manufacturer (none) -> KEMET; Manufacturer Part Number (none) -> C0603C103K4RECTU
- C12, C13: value 1u -> 1uF; footprint Capacitor_SMD:C_0402_1005Metric -> Capacitor_SMD:C_0201_0603Metric; Manufacturer (none) -> Samsung Electro-Mechanics; Manufacturer Part Number (none) -> CL10B105KP8NNNC
- C5: value 10u -> 10uF; Manufacturer (none) -> Taiyo Yuden; Manufacturer Part Number (none) -> LMK107BBJ106MALT
- C7: value 10p -> 10pF; Manufacturer (none) -> KEMET; Manufacturer Part Number (none) -> C0603C100J5GACTU
- D1: value RED -> Green; footprint LED_SMD:LED_0603_1608Metric -> LED_SMD:LED_0402_1005Metric; Manufacturer (none) -> Lite-On Inc.; Manufacturer Part Number (none) -> LTST-C190GKT
Connections:
- net +3.3V: now also C13.2; no longer C13.1
- net GND: now also C12.1, C13.1; no longer C12.2, C13.2
- net at C11.1, FB1.1, U1.9 (VDDA): now also C12.2; no longer C12.1
Other:
- title: (none) -> ADCS-BDOT

Commit message: adcs_board: Few improvements
Parts:
- added C27: 10pF, Capacitor_SMD:C_0402_1005Metric, symbol Device:C
- Y1: value 16 MHz -> 16MHz
Connections:
- net GND: now also C27.2; no longer U1.5 (PD0_OSC_IN), Y1.1
- net HSE_OUT: now reaches C7.1, U1.6 (PD1_OSC_OUT), Y1.3
- new net HSE_IN: C27.1, U1.5 (PD0_OSC_IN), Y1.1
Other:
- note added: "+5V Min 22uF inp/out caps"
- note added: "Oscillator"
- moved on the sheet: C7, D1, R1
